File: console/console01.kicad_pcb (KiCad board)
At the start: 2 copper layers, 50 x 47 mm, 16 parts, among them CON1 7-12V, J1 Video Out, J2 Player 1, J3 Player 2, P1 Color 1, P2 Color 2, P3 Power, P4 Pl2 Pins, P5 Pl1 Pins

Commit message: final version for PCB production
Parts:
- removed the REF*** at (91.5, 87.0)
- added REF***: OSHW-Logo2_7.3x6mm_SilkScreen, Symbols:OSHW-Logo2_7.3x6mm_SilkScreen, F.Cu at (92.5, 84.3)
- added REF***: OSHW-Logo2_7.3x6mm_SilkScreen, Symbols:OSHW-Logo2_7.3x6mm_SilkScreen, B.Cu at (112.0, 95.8)
- P4: footprint Pin_Headers:Pin_Header_Straight_1x04 -> Pin_Headers:Pin_Header_Straight_1x06
- moved P4 2.29 mm to (95.5, 62.2)
Connections:
- J3 pad 1: (no net) -> P2.3
- J3 pad 6: (no net) -> P2.4
- uP1 pad 11: (no net) -> P2.4
- uP1 pad 13: (no net) -> P2.3
- uP1 pad 25: (no net) -> P1.2
- uP1 pad 30: P1.2 -> (no net)
Routing:
- net P2.3: track 0.00 -> 40.5 mm, vias 0 -> 3
- net P2.4: track 0.00 -> 33.6 mm, vias 0 -> 1
- net P1.2: track 16.7 -> 20.0 mm, vias 0 -> 2
- net P2.1: track 16.5 -> 18.1 mm
- net VCC: track 53.3 -> 54.7 mm
- net P2.2: track 35.0 -> 35.5 mm
