File: controller/controller.kicad_pcb (KiCad board)
At the start: 2 copper layers, 45 x 48 mm, 15 parts, among them J1 RJ12, P1 CONN_01X06, SW1 Up, SW2 Right, SW3 Down, SW4 Left

Commit message: final version for PCB production
Parts:
- added RV3: 10k, Potentiometers:Potentiometer_WirePads, F.Cu at (121.9, 126.7)
- added RV4: 10k, added:Potentiometer_Alpha-RV09, F.Cu at (119.4, 110.7)
- moved REF*** 48.9 mm to (147.3, 93.0)
Routing:
- net in2: track 40.9 -> 48.9 mm
- net VCC: track 119.3 -> 124.3 mm
Other:
- board text added: "Arduino VGA Retro Game Console Controller"
- board text removed: "Arduino VGA Retro Game Console"
